Commit message: added rgbd

File: data/robots/mobile.urdf (robot description, URDF)
Before this commit: robot mobile, 4 links, 3 joints
Links:
- added link linkCamera; collision box size=0.02 0.08 0.02; visual box size=0.02 0.05 0.02
Joints:
- added joint jointCamera: type fixed, parent linkBase, child linkCamera, origin xyz=0.175 0.0 0.0 rpy=0 0 0, axis 0 0 1

Commit message: cnn for depth added

File: data/robots/mobile.urdf (robot description, URDF)
Before this commit: robot mobile, 5 links, 4 joints
Links:
- link linkCamera: mass None -> 1.0e-2
